Commit message: Add IMU and MOLA 3D LiDAR baseline

File: src/slam_robot_description/urdf/gazebo.xacro (robot description, xacro)
@@ -3,12 +3,12 @@
   <!-- Contact parameters for the two driven wheels. -->
   <gazebo reference="left_wheel_link">
-    <mu1>1.2</mu1>
-    <mu2>1.2</mu2>
+    <mu1>$(arg left_wheel_friction)</mu1>
+    <mu2>$(arg left_wheel_friction)</mu2>
     <kp>1000000.0</kp>
     <kd>10.0</kd>
   </gazebo>
   <gazebo reference="right_wheel_link">
-    <mu1>1.2</mu1>
-    <mu2>1.2</mu2>
+    <mu1>$(arg right_wheel_friction)</mu1>
+    <mu2>$(arg right_wheel_friction)</mu2>
     <kp>1000000.0</kp>
     <kd>10.0</kd>
@@ -21,5 +21,6 @@
     <kd>10.0</kd>
   </gazebo>
-  <gazebo reference="lidar_link">
+  <xacro:unless value="${'$(arg sensor_variant)' == '3d'}">
+    <gazebo reference="lidar_link">
     <sensor name="lidar_2d" type="gpu_lidar">
       <always_on>true</always_on>
@@ -50,8 +51,70 @@
       </lidar>
     </sensor>
+    </gazebo>
+  </xacro:unless>
+  <xacro:if value="${'$(arg sensor_variant)' == '3d'}">
+    <gazebo reference="lidar_3d_link">
+      <sensor name="lidar_3d" type="gpu_lidar">
+        <always_on>true</always_on>
+        <visualize>false</visualize>
+        <update_rate>$(arg lidar_3d_update_rate)</update_rate>
+        <topic>/lidar_3d</topic>
+        <gz_frame_id>lidar_3d_link</gz_frame_id>
+        <lidar>
+          <scan>
+            <horizontal>
+              <samples>$(arg lidar_3d_horizontal_samples)</samples>
+              <resolution>1.0</resolution>
+              <min_angle>$(arg lidar_3d_horizontal_min_angle)</min_angle>
+              <max_angle>$(arg lidar_3d_horizontal_max_angle)</max_angle>
+            </horizontal>
+            <vertical>
+              <samples>$(arg lidar_3d_vertical_samples)</samples>
+              <resolution>1.0</resolution>
+              <min_angle>$(arg lidar_3d_vertical_min_angle)</min_angle>
+              <max_angle>$(arg lidar_3d_vertical_max_angle)</max_angle>
+            </vertical>
+          </scan>
+          <range>
+            <min>$(arg lidar_3d_minimum_range)</min>
+            <max>$(arg lidar_3d_maximum_range)</max>
+            <resolution>0.01</resolution>
+          </range>
+          <noise>
+            <type>gaussian</type>
+            <mean>0.0</mean>
+            <stddev>$(arg lidar_3d_noise_stddev)</stddev>
+          </noise>
+        </lidar>
+      </sensor>
+    </gazebo>
+  </xacro:if>
+  <gazebo reference="imu_link">
+    <sensor name="imu" type="imu">
+      <always_on>true</always_on>
+      <update_rate>$(arg imu_update_rate)</update_rate>
+      <topic>/imu/data_raw</topic>
+      <gz_frame_id>imu_link</gz_frame_id>
+      <imu>
+        <orientation_reference_frame>
+          <localization>ENU</localization>
+        </orientation_reference_frame>
+        <angular_velocity>
+          <x><noise type="gaussian"><mean>0.0</mean><stddev>$(arg imu_angular_velocity_noise_stddev)</stddev><bias_mean>0.0</bias_mean><bias_stddev>$(arg imu_angular_velocity_bias_stddev)</bias_stddev></noise></x>
+          <y><noise type="gaussian"><mean>0.0</mean><stddev>$(arg imu_angular_velocity_noise_stddev)</stddev><bias_mean>0.0</bias_mean><bias_stddev>$(arg imu_angular_velocity_bias_stddev)</bias_stddev></noise></y>
+          <z><noise type="gaussian"><mean>0.0</mean><stddev>$(arg imu_angular_velocity_noise_stddev)</stddev><bias_mean>0.0</bias_mean><bias_stddev>$(arg imu_angular_velocity_bias_stddev)</bias_stddev></noise></z>
+        </angular_velocity>
+        <linear_acceleration>
+          <x><noise type="gaussian"><mean>0.0</mean><stddev>$(arg imu_linear_acceleration_noise_stddev)</stddev><bias_mean>0.0</bias_mean><bias_stddev>$(arg imu_linear_acceleration_bias_stddev)</bias_stddev></noise></x>
+          <y><noise type="gaussian"><mean>0.0</mean><stddev>$(arg imu_linear_acceleration_noise_stddev)</stddev><bias_mean>0.0</bias_mean><bias_stddev>$(arg imu_linear_acceleration_bias_stddev)</bias_stddev></noise></y>
+          <z><noise type="gaussian"><mean>0.0</mean><stddev>$(arg imu_linear_acceleration_noise_stddev)</stddev><bias_mean>0.0</bias_mean><bias_stddev>$(arg imu_linear_acceleration_bias_stddev)</bias_stddev></noise></z>
+        </linear_acceleration>
+      </imu>
+    </sensor>
   </gazebo>
   <gazebo>
     <self_collide>false</self_collide>
-    <plugin
+    <xacro:macro name="diff_drive_plugin" params="odom_topic tf_topic">
+      <plugin
       filename="gz-sim-diff-drive-system"
       name="gz::sim::systems::DiffDrive">
@@ -62,6 +125,6 @@
       <wheel_radius>${wheel_radius}</wheel_radius>
       <topic>/cmd_vel</topic>
-      <odom_topic>/odom</odom_topic>
-      <tf_topic>/model/slam_robot/tf</tf_topic>
+      <odom_topic>${odom_topic}</odom_topic>
+      <tf_topic>${tf_topic}</tf_topic>
       <frame_id>odom</frame_id>
       <child_frame_id>base_footprint</child_frame_id>
@@ -80,5 +143,16 @@
       <max_angular_acceleration>2.00</max_angular_acceleration>
       <min_angular_acceleration>-2.00</min_angular_acceleration>
-    </plugin>
+      </plugin>
+    </xacro:macro>
+    <xacro:if value="${'$(arg odometry_mode)' == 'wheel_imu'}">
+      <xacro:diff_drive_plugin
+        odom_topic="/wheel/odom"
+        tf_topic="/model/slam_robot/wheel_tf"/>
+    </xacro:if>
+    <xacro:unless value="${'$(arg odometry_mode)' == 'wheel_imu'}">
+      <xacro:diff_drive_plugin
+        odom_topic="/odom"
+        tf_topic="/model/slam_robot/tf"/>
+    </xacro:unless>
     <plugin
       filename="gz-sim-joint-state-publisher-system"

File: src/slam_robot_description/urdf/slam_robot.urdf.xacro (robot description, xacro)
@@ -1,4 +1,29 @@
 <?xml version="1.0"?>
 <robot name="slam_robot" xmlns:xacro="http://www.ros.org/wiki/xacro">
+  <xacro:arg name="sensor_variant" default="2d"/>
+  <xacro:arg name="odometry_mode" default="wheel"/>
+  <xacro:arg name="left_wheel_friction" default="1.2"/>
+  <xacro:arg name="right_wheel_friction" default="1.2"/>
+  <xacro:arg name="lidar_3d_x" default="-0.07"/>
+  <xacro:arg name="lidar_3d_y" default="0.0"/>
+  <xacro:arg name="lidar_3d_z" default="0.18"/>
+  <xacro:arg name="lidar_3d_roll" default="0.0"/>
+  <xacro:arg name="lidar_3d_pitch" default="0.0"/>
+  <xacro:arg name="lidar_3d_yaw" default="0.0"/>
+  <xacro:arg name="lidar_3d_horizontal_samples" default="720"/>
+  <xacro:arg name="lidar_3d_horizontal_min_angle" default="-3.141592653589793"/>
+  <xacro:arg name="lidar_3d_horizontal_max_angle" default="3.1328660073298216"/>
+  <xacro:arg name="lidar_3d_vertical_samples" default="16"/>
+  <xacro:arg name="lidar_3d_vertical_min_angle" default="-0.2617993877991494"/>
+  <xacro:arg name="lidar_3d_vertical_max_angle" default="0.2617993877991494"/>
+  <xacro:arg name="lidar_3d_update_rate" default="10.0"/>
+  <xacro:arg name="lidar_3d_minimum_range" default="0.20"/>
+  <xacro:arg name="lidar_3d_maximum_range" default="20.0"/>
+  <xacro:arg name="lidar_3d_noise_stddev" default="0.01"/>
+  <xacro:arg name="imu_update_rate" default="100.0"/>
+  <xacro:arg name="imu_angular_velocity_noise_stddev" default="0.002"/>
+  <xacro:arg name="imu_angular_velocity_bias_stddev" default="0.0002"/>
+  <xacro:arg name="imu_linear_acceleration_noise_stddev" default="0.02"/>
+  <xacro:arg name="imu_linear_acceleration_bias_stddev" default="0.005"/>
   <xacro:include filename="$(find slam_robot_description)/urdf/materials.xacro"/>
   <xacro:include filename="$(find slam_robot_description)/urdf/inertial_macros.xacro"/>
@@ -30,4 +55,15 @@
   <xacro:property name="lidar_mount_height" value="0.10"/>
   <xacro:property name="lidar_mount_mass" value="0.12"/>
+  <!-- The 2D and 3D LiDAR variants are mutually exclusive. -->
+  <xacro:property name="lidar_3d_mount_radius" value="0.028"/>
+  <xacro:property name="lidar_3d_mount_height" value="0.085"/>
+  <xacro:property name="lidar_3d_mount_mass" value="0.10"/>
+  <xacro:property name="lidar_3d_radius" value="0.055"/>
+  <xacro:property name="lidar_3d_height" value="0.07"/>
+  <xacro:property name="lidar_3d_mass" value="0.32"/>
+  <xacro:property name="imu_length" value="0.04"/>
+  <xacro:property name="imu_width" value="0.03"/>
+  <xacro:property name="imu_height" value="0.015"/>
+  <xacro:property name="imu_mass" value="0.02"/>
   <link name="base_footprint"/>
   <link name="base_link">
@@ -122,5 +158,29 @@
       rpy="0 0 0"/>
   </joint>
-  <link name="lidar_mount_link">
+  <link name="imu_link">
+    <visual>
+      <geometry>
+        <box size="${imu_length} ${imu_width} ${imu_height}"/>
+      </geometry>
+      <material name="accent_orange"/>
+    </visual>
+    <inertial>
+      <mass value="${imu_mass}"/>
+      <inertia
+        ixx="${imu_mass * (imu_width * imu_width + imu_height * imu_height) / 12.0}"
+        ixy="0.0"
+        ixz="0.0"
+        iyy="${imu_mass * (imu_length * imu_length + imu_height * imu_height) / 12.0}"
+        iyz="0.0"
+        izz="${imu_mass * (imu_length * imu_length + imu_width * imu_width) / 12.0}"/>
+    </inertial>
+  </link>
+  <joint name="imu_joint" type="fixed">
+    <parent link="base_link"/>
+    <child link="imu_link"/>
+    <origin xyz="0 0 0" rpy="0 0 0"/>
+  </joint>
+  <xacro:unless value="${'$(arg sensor_variant)' == '3d'}">
+    <link name="lidar_mount_link">
     <visual>
       <geometry>
@@ -138,6 +198,6 @@
       radius="${lidar_mount_radius}"
       length="${lidar_mount_height}"/>
-  </link>
-  <joint name="lidar_mount_joint" type="fixed">
+    </link>
+    <joint name="lidar_mount_joint" type="fixed">
     <parent link="base_link"/>
     <child link="lidar_mount_link"/>
@@ -145,6 +205,6 @@
       xyz="${-drive_axle_offset} 0 ${base_height / 2.0 + lidar_mount_height / 2.0}"
       rpy="0 0 0"/>
-  </joint>
-  <link name="lidar_link">
+    </joint>
+    <link name="lidar_link">
     <visual>
       <geometry>
@@ -162,10 +222,61 @@
       radius="${lidar_radius}"
       length="${lidar_height}"/>
-  </link>
-  <joint name="lidar_joint" type="fixed">
-    <parent link="lidar_mount_link"/>
-    <child link="lidar_link"/>
-    <origin xyz="0 0 ${(lidar_mount_height + lidar_height) / 2.0}" rpy="0 0 0"/>
-  </joint>
+    </link>
+    <joint name="lidar_joint" type="fixed">
+      <parent link="lidar_mount_link"/>
+      <child link="lidar_link"/>
+      <origin xyz="0 0 ${(lidar_mount_height + lidar_height) / 2.0}" rpy="0 0 0"/>
+    </joint>
+  </xacro:unless>
+  <xacro:if value="${'$(arg sensor_variant)' == '3d'}">
+    <link name="lidar_3d_mount_link">
+      <visual>
+        <geometry>
+          <cylinder radius="${lidar_3d_mount_radius}" length="${lidar_3d_mount_height}"/>
+        </geometry>
+        <material name="accent_orange"/>
+      </visual>
+      <collision>
+        <geometry>
+          <cylinder radius="${lidar_3d_mount_radius}" length="${lidar_3d_mount_height}"/>
+        </geometry>
+      </collision>
+      <xacro:cylinder_inertial
+        mass="${lidar_3d_mount_mass}"
+        radius="${lidar_3d_mount_radius}"
+        length="${lidar_3d_mount_height}"/>
+    </link>
+    <joint name="lidar_3d_mount_joint" type="fixed">
+      <parent link="base_link"/>
+      <child link="lidar_3d_mount_link"/>
+      <origin
+        xyz="$(arg lidar_3d_x) $(arg lidar_3d_y) ${float('$(arg lidar_3d_z)') - (lidar_3d_mount_height + lidar_3d_height) / 2.0}"
+        rpy="$(arg lidar_3d_roll) $(arg lidar_3d_pitch) $(arg lidar_3d_yaw)"/>
+    </joint>
+    <link name="lidar_3d_link">
+      <visual>
+        <geometry>
+          <cylinder radius="${lidar_3d_radius}" length="${lidar_3d_height}"/>
+        </geometry>
+        <material name="sensor_gray"/>
+      </visual>
+      <collision>
+        <geometry>
+          <cylinder radius="${lidar_3d_radius}" length="${lidar_3d_height}"/>
+        </geometry>
+      </collision>
+      <xacro:cylinder_inertial
+        mass="${lidar_3d_mass}"
+        radius="${lidar_3d_radius}"
+        length="${lidar_3d_height}"/>
+    </link>
+    <joint name="lidar_3d_joint" type="fixed">
+      <parent link="lidar_3d_mount_link"/>
+      <child link="lidar_3d_link"/>
+      <origin
+        xyz="0 0 ${(lidar_3d_mount_height + lidar_3d_height) / 2.0}"
+        rpy="0 0 0"/>
+    </joint>
+  </xacro:if>
   <xacro:include filename="$(find slam_robot_description)/urdf/gazebo.xacro"/>
 </robot>

Commit message: Add RGB-D simulation sensor foundation

File: src/slam_robot_description/urdf/gazebo.xacro (robot description, xacro)
@@ -90,4 +90,26 @@
     </gazebo>
   </xacro:if>
+  <xacro:if value="${'$(arg camera_variant)' == 'rgbd'}">
+    <gazebo reference="camera_link">
+      <sensor name="rgbd_camera" type="rgbd_camera">
+        <always_on>true</always_on>
+        <visualize>false</visualize>
+        <update_rate>$(arg rgbd_update_rate)</update_rate>
+        <topic>/camera</topic>
+        <camera>
+          <horizontal_fov>$(arg rgbd_horizontal_fov)</horizontal_fov>
+          <image>
+            <width>$(arg rgbd_width)</width>
+            <height>$(arg rgbd_height)</height>
+          </image>
+          <clip>
+            <near>$(arg rgbd_minimum_depth)</near>
+            <far>$(arg rgbd_maximum_depth)</far>
+          </clip>
+          <optical_frame_id>camera_optical_frame</optical_frame_id>
+        </camera>
+      </sensor>
+    </gazebo>
+  </xacro:if>
   <gazebo reference="imu_link">
     <sensor name="imu" type="imu">

File: src/slam_robot_description/urdf/slam_robot.urdf.xacro (robot description, xacro)
@@ -2,4 +2,5 @@
 <robot name="slam_robot" xmlns:xacro="http://www.ros.org/wiki/xacro">
   <xacro:arg name="sensor_variant" default="2d"/>
+  <xacro:arg name="camera_variant" default="none"/>
   <xacro:arg name="odometry_mode" default="wheel"/>
   <xacro:arg name="left_wheel_friction" default="1.2"/>
@@ -21,4 +22,10 @@
   <xacro:arg name="lidar_3d_maximum_range" default="20.0"/>
   <xacro:arg name="lidar_3d_noise_stddev" default="0.01"/>
+  <xacro:arg name="rgbd_width" default="640"/>
+  <xacro:arg name="rgbd_height" default="480"/>
+  <xacro:arg name="rgbd_update_rate" default="30.0"/>
+  <xacro:arg name="rgbd_horizontal_fov" default="1.2217304763960306"/>
+  <xacro:arg name="rgbd_minimum_depth" default="0.20"/>
+  <xacro:arg name="rgbd_maximum_depth" default="6.0"/>
   <xacro:arg name="imu_update_rate" default="100.0"/>
   <xacro:arg name="imu_angular_velocity_noise_stddev" default="0.002"/>
@@ -66,4 +73,19 @@
   <xacro:property name="imu_height" value="0.015"/>
   <xacro:property name="imu_mass" value="0.02"/>
+  <!--
+    The RGB-D optical centre is flush with the chassis front face. The housing
+    extends rearward, so enabling the camera does not enlarge the existing
+    Nav2 footprint. Its top remains below the lowest -15 degree 3D LiDAR ray.
+  -->
+  <xacro:property name="camera_x" value="0.155"/>
+  <xacro:property name="camera_z" value="0.09"/>
+  <xacro:property name="camera_body_length" value="0.03"/>
+  <xacro:property name="camera_body_width" value="0.14"/>
+  <xacro:property name="camera_body_height" value="0.04"/>
+  <xacro:property name="camera_body_mass" value="0.09"/>
+  <xacro:property name="camera_mount_length" value="0.03"/>
+  <xacro:property name="camera_mount_width" value="0.04"/>
+  <xacro:property name="camera_mount_height" value="0.015"/>
+  <xacro:property name="camera_mount_mass" value="0.03"/>
   <link name="base_footprint"/>
   <link name="base_link">
@@ -181,4 +203,71 @@
     <origin xyz="0 0 0" rpy="0 0 0"/>
   </joint>
+  <xacro:if value="${'$(arg camera_variant)' == 'rgbd'}">
+    <link name="camera_mount_link">
+      <visual>
+        <geometry>
+          <box size="${camera_mount_length} ${camera_mount_width} ${camera_mount_height}"/>
+        </geometry>
+        <material name="accent_orange"/>
+      </visual>
+      <collision>
+        <geometry>
+          <box size="${camera_mount_length} ${camera_mount_width} ${camera_mount_height}"/>
+        </geometry>
+      </collision>
+      <xacro:box_inertial
+        mass="${camera_mount_mass}"
+        length="${camera_mount_length}"
+        width="${camera_mount_width}"
+        height="${camera_mount_height}"/>
+    </link>
+    <joint name="camera_mount_joint" type="fixed">
+      <parent link="base_link"/>
+      <child link="camera_mount_link"/>
+      <origin
+        xyz="${camera_x - camera_body_length} 0 ${base_height / 2.0 + camera_mount_height / 2.0}"
+        rpy="0 0 0"/>
+    </joint>
+    <link name="camera_link">
+      <visual>
+        <origin xyz="${-camera_body_length / 2.0} 0 0" rpy="0 0 0"/>
+        <geometry>
+          <box size="${camera_body_length} ${camera_body_width} ${camera_body_height}"/>
+        </geometry>
+        <material name="sensor_gray"/>
+      </visual>
+      <collision>
+        <origin xyz="${-camera_body_length / 2.0} 0 0" rpy="0 0 0"/>
+        <geometry>
+          <box size="${camera_body_length} ${camera_body_width} ${camera_body_height}"/>
+        </geometry>
+      </collision>
+      <inertial>
+        <mass value="${camera_body_mass}"/>
+        <origin xyz="${-camera_body_length / 2.0} 0 0" rpy="0 0 0"/>
+        <inertia
+          ixx="${camera_body_mass * (camera_body_width * camera_body_width + camera_body_height * camera_body_height) / 12.0}"
+          ixy="0.0"
+          ixz="0.0"
+          iyy="${camera_body_mass * (camera_body_length * camera_body_length + camera_body_height * camera_body_height) / 12.0}"
+          iyz="0.0"
+          izz="${camera_body_mass * (camera_body_length * camera_body_length + camera_body_width * camera_body_width) / 12.0}"/>
+      </inertial>
+    </link>
+    <joint name="camera_joint" type="fixed">
+      <parent link="camera_mount_link"/>
+      <child link="camera_link"/>
+      <origin
+        xyz="${camera_body_length} 0 ${camera_z - (base_height / 2.0 + camera_mount_height / 2.0)}"
+        rpy="0 0 0"/>
+    </joint>
+    <link name="camera_optical_frame"/>
+    <joint name="camera_optical_joint" type="fixed">
+      <parent link="camera_link"/>
+      <child link="camera_optical_frame"/>
+      <!-- REP-103 camera frame (x forward) to optical frame (z forward). -->
+      <origin xyz="0 0 0" rpy="${-pi / 2.0} 0 ${-pi / 2.0}"/>
+    </joint>
+  </xacro:if>
   <xacro:unless value="${'$(arg sensor_variant)' == '3d'}">
     <link name="lidar_mount_link">
